File: template.kicad_pcb (KiCad board)
At the start: 4 copper layers, 63 x 35.6 mm, 47 parts, among them J1 Barrel_Jack_Switch, J2 USB_B, J3 P1, J4 2x2M, J5 ICSP1, J6 P2, U1 ATmega8U2-AU, Y1 16MHz

Commit message: 测试整合CI文件
Other:
- board text added: "variants template"
- board text removed: "KiBot variants example Not a real life board"
Changed lines of the file:
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@@
     (rev "${git_hash}")
     (company "Instituto Nacional de Tecnología Industrial")
-    (comment 4 "An example of KiBot variants")
+    (comment 4 "KiBot variants template")
   )
   (layers
@@
   (gr_line (start 119 65.7) (end 119 101.3) (layer "Edge.Cuts") (width 0.05))
   (gr_line (start 182 65.7) (end 119 65.7) (layer "Edge.Cuts") (width 0.05))
-  (gr_text "KiBot variants example\nNot a real life board" (at 128.7272 88.011) (layer "B.SilkS")
+  (gr_text "variants template" (at 128.7272 88.011) (layer "B.SilkS")
     (effects (font (size 1 1) (thickness 0.15)) (justify mirror))
   )
