File: template.kicad_sch (KiCad schematic)
At the start: 47 parts, among them J1 Barrel_Jack_Switch, J2 USB_B, J3 P1, J4 2x2M, J5 ICSP1, J6 P2, U1 ATmega8U2-AU, Y1 16MHz

Commit message: 测试整合CI文件
Other:
- note added: "variants template"
- note removed: "KiBot variants example Not a real life board"
Changed lines of the file:
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@@
   (title_block
     (title "Arduino UNO programmer")
-    (date "2020-09-09")
+    (date "2022-07-23")
     (rev "r1")
     (company "Arduino")
@@
   )
   (text "This logo has a REF starting with #\nWon't be passed to the PCB"
-    (at 105.41 189.23 0)
+    (at 111.76 184.15 0)
     (effects (font (size 2.0066 2.0066)) (justify left bottom))
   )
-  (text "KiBot variants example\nNot a real life board" (at 13.97 25.4 0)
-    (effects (font (size 3.9878 3.9878)) (justify left bottom))
+  (text "variants template" (at 15.24 19.05 0)
+    (effects (font (size 3.9878 3.9878) (thickness 0.7976) bold) (justify left bottom))
   )
   (label "RESET2" (at 121.92 72.39 0)
@@
     (pin "1")
   )
-  (symbol (lib_id "Graphic:SYM_Magnet_Large") (at 127 176.53 0) (unit 1)
-    (in_bom yes) (on_board yes)
-    (property "Reference" "#SYM1" (id 0) (at 127 171.45 0)
-      (effects (font (size 1.27 1.27)) hide)
-    )
-    (property "Value" "SYM_Magnet_Large" (id 1) (at 127 182.88 0)
-      (effects (font (size 1.27 1.27)) hide)
-    )
-    (property "Footprint" "" (id 2) (at 127 181.61 0)
-      (effects (font (size 1.27 1.27)) hide)
-    )
-    (property "Datasheet" "~" (id 3) (at 127.762 181.61 0)
-      (effects (font (size 1.27 1.27)) hide)
-    )
+  (symbol (lib_id "Graphic:SYM_Magnet_Large") (at 135.89 168.91 0) (unit 1)
+    (in_bom yes) (on_board yes)
+    (property "Reference" "#SYM1" (id 0) (at 135.89 163.83 0)
+      (effects (font (size 1.27 1.27)) hide)
+    )
+    (property "Value" "SYM_Magnet_Large" (id 1) (at 135.89 175.26 0)
+      (effects (font (size 1.27 1.27)) hide)
+    )
+    (property "Footprint" "" (id 2) (at 135.89 173.99 0)
+      (effects (font (size 1.27 1.27)) hide)
+    )
+    (property "Datasheet" "~" (id 3) (at 136.652 173.99 0)
+      (effects (font (size 1.27 1.27)) hide)
+    )
